File: Hardware/DomoMod.brd (EAGLE design)
At the start: 80 x 30 mm, 47 parts, among them Q1 BSS138, Q2 BSS138, T1 MMBT2222A, U1 NCS36000, U2 CCS811, U3 BME280, U4 PIR

Commit message: Update
Parts:
- removed JP7: (no value), pinhead:1X03
- removed JP8: (no value), pinhead:1X04
- removed R18, R19: 10k, SparkFun-Resistors:0603
- added JP1, JP2: (no value), pinhead:1X02
- added POT1, POT2: 1M, openPIR-temp:TRIMPOT-TC33X
- JP5: device pinhead:1X02 -> pinhead:1X03
- JP6: device pinhead:1X02 -> pinhead:1X04
- R1: value 10k -> 1k
- R11: value 560k -> 10k; device openPIR-temp:0603 -> SparkFun-Resistors:0603
- R12: value 10k -> 43k
- R13: value 1M -> 51k; device openPIR-temp:TRIMPOT-TC33X -> openPIR-temp:0603
- R14: value 1M -> 100k; device openPIR-temp:TRIMPOT-TC33X -> SparkFun-Resistors:0603
- R15: value 51k -> 100k; device openPIR-temp:0603 -> SparkFun-Resistors:0603
- R16: value 1k -> 100k
- R17: value 10k -> 560k; device SparkFun-Resistors:0603 -> openPIR-temp:0603
- R2: value 10k -> 4.7k
- R5: value 4.7k -> 10k
- R6, R7, R8: value 100k -> 10k
- R9: value 43k -> 10k
- moved R1 65.0 mm to (68.0, 19.5), turned to 0 degrees
- moved R8 53.1 mm to (71.0, 12.5), turned to 180 degrees
- moved R7 50.3 mm to (71.0, 15.5), turned to 180 degrees
- moved R16 48.3 mm to (21.5, 6.50)
- moved R14 43.2 mm to (18.0, 10.0)
- moved R15 31.3 mm to (10.0, 10.0), turned to 270 degrees
- moved R12 18.6 mm to (53.5, 6.00)
- moved R17 18.2 mm to (54.0, 22.0)
- moved R9 18.0 mm to (71.0, 10.0)
- moved JP6 17.4 mm to (73.7, 27.2), turned to 0 degrees
- moved R5 15.6 mm to (3.00, 17.5), turned to 90 degrees
- moved R2 15.1 mm to (14.0, 6.50), turned to 180 degrees
- moved JP5 10.3 mm to (75.0, 23.2), turned to 0 degrees
- moved R13 9.90 mm to (39.5, 20.5), turned to 0 degrees
- moved R11 9.00 mm to (63.0, 22.0)
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- renumbered SV2 to SV1
Connections:
- net !RST: now also R2.1; no longer R5.1
- net !WAKE: now also R14.2; no longer R8.2
- net 3.3V: now also R15.2, R16.2, R2.2; no longer R1.2, R6.2, R7.2
- net A1: now also JP2.2, R7.2; no longer JP4.2, R17.2
- net A2: now also POT1.1; no longer R13.1
- net A3: now also JP4.2, R9.2; no longer JP6.2, R19.2
- net A4: now also JP3.2, R8.2; no longer JP5.2, R18.2
- net CCS811_ADDR: now also R15.1; no longer R6.1
- net D2: now also JP6.2, R4.1; no longer JP8.2, R2.1
- net D3: now also JP6.1, R6.1; no longer JP8.1, R4.1
- net D5: now also JP5.1; no longer JP7.1
- net D6: now also R1.2; no longer R16.2
- net D7: now also JP4.1; no longer JP6.1
- net GND: now also JP5.3, JP6.4, R12.1, R14.1, R7.1; no longer JP7.3, JP8.4, R17.1, R18.1, R19.1
- net N$1: now also R12.2; no longer R9.2
- net N$10: now also R1.1; no longer R16.1
- net N$11: now also POT2.1, R13.2; no longer R14.1, R15.2
- net N$4: now also R11.1; no longer R12.1
- net N$5: now also R17.1; no longer R11.1
- net N$6: now also R17.2; no longer R11.2
- net N$7: now also POT1.2, POT1.3, R11.2; no longer R12.2, R13.2, R13.3
- net N$8: now also R13.1; no longer R15.1
- net N$9: now also JP1.2; no longer JP3.2
- net SCL: now also R5.1; no longer R3.1
- net SDA: now also R3.1; no longer R1.1
- net SDO/ADR: now also R16.1; no longer R7.1
- net VCC: now also JP1.1, JP2.1, JP5.2, JP6.3, POT2.2, POT2.3, R6.2; no longer JP4.1, JP5.1, JP7.2, JP8.3, R14.2, R14.3, R2.2
